Commit message: reversed comments

File: cartographer_config/lidar_stick.urdf (robot description, URDF)
Before this commit: robot cartographer_backpack_3d, 4 links, 3 joints
Links:
- removed link horizontal_vlp16_link
- removed link imu_link
- removed link vertical_vlp16_link
- added link gx5_link; visual box size=0.06 0.04 0.02
- added link velodyne; visual cylinder length=0.07 radius=0.05
Joints:
- removed joint horizontal_vlp16_link_joint
- removed joint imu_link_joint
- removed joint vertical_vlp16_link_joint
- added joint gx5_link_joint: type fixed, parent base_link, child gx5_link, origin xyz=0 0 0 rpy=3.1416 0 0
- added joint velodyne_joint: type fixed, parent base_link, child velodyne, origin xyz=0.00 0. 0.2 rpy=0. 0 0

Commit message: testing changes to imu orientation, slam seems more sensitive to motion rather than imu rotation

File: cartographer_config/lidar_stick.urdf (robot description, URDF)
Before this commit: robot cartographer_backpack_3d, 3 links, 2 joints
Joints:
- joint gx5_link_joint: origin xyz=0 0 0 rpy=3.1416 0 0 -> xyz=0 0 0 rpy=0 -1.57079632679 0
- joint velodyne_joint: origin xyz=0.00 0. 0.2 rpy=0. 0 0 -> xyz=0.1 0 0.1 rpy=0. 0 0

Commit message: Update lidar_stick.urdf

File: cartographer_config/lidar_stick.urdf (robot description, URDF)
Before this commit: robot cartographer_backpack_3d, 3 links, 2 joints
Links:
- link gx5_link: geometry visual box size=0.036 0.024 0.0111
- link velodyne: geometry visual cylinder length=0.0869 radius=0.05
Joints:
- joint velodyne_joint: origin xyz=0.1 0 0.1 rpy=0. 0 0 -> xyz=0.030988 0 0.087378 rpy=0. 0 0

Commit message: Update lidar_stick.urdf

File: cartographer_config/lidar_stick.urdf (robot description, URDF)
Before this commit: robot cartographer_backpack_3d, 3 links, 2 joints
Joints:
- joint velodyne_joint: origin xyz=0.030988 0 0.087378 rpy=0. 0 0 -> xyz=0.030988 0 -0.087378 rpy=0. 0 0

Commit message: Update lidar_stick.urdf

File: cartographer_config/lidar_stick.urdf (robot description, URDF)
Before this commit: robot cartographer_backpack_3d, 3 links, 2 joints
Joints:
- joint velodyne_joint: origin xyz=0.030988 0 -0.087378 rpy=0. 0 0 -> xyz=-0.030988 0 0.087378 rpy=0. 0 0

Commit message: Update lidar_stick.urdf

File: cartographer_config/lidar_stick.urdf (robot description, URDF)
Before this commit: robot cartographer_backpack_3d, 3 links, 2 joints
Joints:
- joint gx5_link_joint: origin xyz=0 0 0 rpy=0 -1.57079632679 0 -> xyz=0 0 0 rpy=0 1.57079632679 0
- joint velodyne_joint: origin xyz=-0.030988 0 0.087378 rpy=0. 0 0 -> xyz=0.030988 0 0.087378 rpy=0. 0 0

Commit message: Update lidar_stick.urdf

File: cartographer_config/lidar_stick.urdf (robot description, URDF)
Before this commit: robot cartographer_backpack_3d, 3 links, 2 joints
Joints:
- joint gx5_link_joint: origin xyz=0 0 0 rpy=0 1.57079632679 0 -> xyz=0 0 0 rpy=0 -1.57079632679 0
- joint velodyne_joint: origin xyz=0.030988 0 0.087378 rpy=0. 0 0 -> xyz=0.030988 0 0.087378 rpy=0. 3.14159265358979 0

Commit message: Update lidar_stick.urdf

File: cartographer_config/lidar_stick.urdf (robot description, URDF)
Before this commit: robot cartographer_backpack_3d, 3 links, 2 joints
Joints:
- joint velodyne_joint: origin xyz=0.030988 0 0.087378 rpy=0. 3.14159265358979 0 -> xyz=0.030988 0 0.087378 rpy=0. 0 0

Commit message: Update lidar_stick.urdf

File: cartographer_config/lidar_stick.urdf (robot description, URDF)
Before this commit: robot cartographer_backpack_3d, 3 links, 2 joints
Joints:
- joint velodyne_joint: origin xyz=0.030988 0 0.087378 rpy=0. 0 0 -> xyz=0.030988 0 0.087378 rpy=0. 0 3.1415926535

Commit message: Update lidar_stick.urdf

File: cartographer_config/lidar_stick.urdf (robot description, URDF)
Before this commit: robot cartographer_backpack_3d, 3 links, 2 joints
Joints:
- joint velodyne_joint: origin xyz=0.030988 0 0.087378 rpy=0. 0 3.1415926535 -> xyz=0.030988 0 0.087378 rpy=0. 0 1.57079632679

Commit message: Update lidar_stick.urdf

File: cartographer_config/lidar_stick.urdf (robot description, URDF)
Before this commit: robot cartographer_backpack_3d, 3 links, 2 joints
Joints:
- joint velodyne_joint: origin xyz=0.030988 0 0.087378 rpy=0. 0 1.57079632679 -> xyz=0.030988 0 0.087378 rpy=0. 0 0

Commit message: Update lidar_stick.urdf

File: cartographer_config/lidar_stick.urdf (robot description, URDF)
Before this commit: robot cartographer_backpack_3d, 3 links, 2 joints
Joints:
- joint gx5_link_joint: origin xyz=0 0 0 rpy=0 -1.57079632679 0 -> xyz=0 0 0 rpy=0 -1.57079632679 3.14159265358979

Commit message: Update lidar_stick.urdf

File: cartographer_config/lidar_stick.urdf (robot description, URDF)
Before this commit: robot cartographer_backpack_3d, 3 links, 2 joints
Joints:
- joint gx5_link_joint: origin xyz=0 0 0 rpy=0 -1.57079632679 3.14159265358979 -> xyz=0 0 0 rpy=0 -1.57079632679 0
- joint velodyne_joint: origin xyz=0.030988 0 0.087378 rpy=0. 0 0 -> xyz=-0.030988 0 0.087378 rpy=0. 0 0

Commit message: Update lidar_stick.urdf

File: cartographer_config/lidar_stick.urdf (robot description, URDF)
Before this commit: robot cartographer_backpack_3d, 3 links, 2 joints
Joints:
- joint velodyne_joint: origin xyz=-0.030988 0 0.087378 rpy=0. 0 0 -> xyz=0.030988 0 0.087378 rpy=0. 0 0

Commit message: Update lidar_stick.urdf

File: cartographer_config/lidar_stick.urdf (robot description, URDF)
Before this commit: robot cartographer_backpack_3d, 3 links, 2 joints
Joints:
- joint velodyne_joint: origin xyz=0.030988 0 0.087378 rpy=0. 0 0 -> xyz=0.030988 0 0.087378 rpy=0. 3.14159265358979 0

Commit message: Update lidar_stick.urdf

File: cartographer_config/lidar_stick.urdf (robot description, URDF)
Before this commit: robot cartographer_backpack_3d, 3 links, 2 joints
Joints:
- joint gx5_link_joint: origin xyz=0 0 0 rpy=0 -1.57079632679 0 -> xyz=0 0 0 rpy=0 1.57079632679 0
- joint velodyne_joint: origin xyz=0.030988 0 0.087378 rpy=0. 3.14159265358979 0 -> xyz=0.030988 0 0.087378 rpy=0. 0 0

Commit message: Update lidar_stick.urdf

File: cartographer_config/lidar_stick.urdf (robot description, URDF)
Before this commit: robot cartographer_backpack_3d, 3 links, 2 joints
Joints:
- joint velodyne_joint: origin xyz=0.030988 0 0.087378 rpy=0. 0 0 -> xyz=-0.030988 0 -0.087378 rpy=0. 0 0

Commit message: Update lidar_stick.urdf

File: cartographer_config/lidar_stick.urdf (robot description, URDF)
Before this commit: robot cartographer_backpack_3d, 3 links, 2 joints
Joints:
- joint gx5_link_joint: origin xyz=0 0 0 rpy=0 1.57079632679 0 -> xyz=0 0 0 rpy=0 -1.57079632679 3.14159265358979
- joint velodyne_joint: origin xyz=-0.030988 0 -0.087378 rpy=0. 0 0 -> xyz=0.030988 0 0.087378 rpy=0. 0 0

Commit message: Update lidar_stick.urdf

File: cartographer_config/lidar_stick.urdf (robot description, URDF)
Before this commit: robot cartographer_backpack_3d, 3 links, 2 joints
Joints:
- joint gx5_link_joint: origin xyz=0 0 0 rpy=0 -1.57079632679 3.14159265358979 -> xyz=0 0 0 rpy=0 1.57079632679 3.14159265358979
- joint velodyne_joint: origin xyz=0.030988 0 0.087378 rpy=0. 0 0 -> xyz=-0.030988 0 -0.087378 rpy=0. 0 0

Commit message: Update lidar_stick.urdf

File: cartographer_config/lidar_stick.urdf (robot description, URDF)
Before this commit: robot cartographer_backpack_3d, 3 links, 2 joints
Joints:
- joint velodyne_joint: origin xyz=-0.030988 0 -0.087378 rpy=0. 0 0 -> xyz=-0.030988 0 0.087378 rpy=0. 0 0

Commit message: Update lidar_stick.urdf

File: cartographer_config/lidar_stick.urdf (robot description, URDF)
Before this commit: robot cartographer_backpack_3d, 3 links, 2 joints
Joints:
- joint velodyne_joint: origin xyz=-0.030988 0 0.087378 rpy=0. 0 0 -> xyz=0.030988 0 -0.087378 rpy=0. 0 0

Commit message: Update lidar_stick.urdf

File: cartographer_config/lidar_stick.urdf (robot description, URDF)
Before this commit: robot cartographer_backpack_3d, 3 links, 2 joints
Joints:
- joint gx5_link_joint: origin xyz=0 0 0 rpy=0 1.57079632679 3.14159265358979 -> xyz=0 0 0 rpy=3.14159265358979 -1.57079632679 0
- joint velodyne_joint: origin xyz=0.030988 0 -0.087378 rpy=0. 0 0 -> xyz=0.030988 0 0.087378 rpy=0. 0 0

Commit message: Update lidar_stick.urdf

File: cartographer_config/lidar_stick.urdf (robot description, URDF)
Before this commit: robot cartographer_backpack_3d, 3 links, 2 joints
Joints:
- joint gx5_link_joint: origin xyz=0 0 0 rpy=3.14159265358979 -1.57079632679 0 -> xyz=0 0 0 rpy=3.14159265358979 1.57079632679 0
- joint velodyne_joint: origin xyz=0.030988 0 0.087378 rpy=0. 0 0 -> xyz=-0.030988 0 -0.087378 rpy=0. 0 0

Commit message: Update lidar_stick.urdf

File: cartographer_config/lidar_stick.urdf (robot description, URDF)
Before this commit: robot cartographer_backpack_3d, 3 links, 2 joints
Joints:
- joint gx5_link_joint: origin xyz=0 0 0 rpy=3.14159265358979 1.57079632679 0 -> xyz=0 0 0 rpy=3.14159265358979 -1.57079632679 0

Commit message: Update lidar_stick.urdf

File: cartographer_config/lidar_stick.urdf (robot description, URDF)
Before this commit: robot cartographer_backpack_3d, 3 links, 2 joints
Joints:
- joint gx5_link_joint: origin xyz=0 0 0 rpy=0 -1.57079632679 0 -> xyz=0 0 0 rpy=0 0 0

Commit message: Update lidar_stick.urdf

File: cartographer_config/lidar_stick.urdf (robot description, URDF)
Before this commit: robot cartographer_backpack_3d, 3 links, 2 joints
Joints:
- joint gx5_link_joint: origin xyz=0 0 0 rpy=0 0 0 -> xyz=0 0 0 rpy=-1.57079632. 0 0

Commit message: Update lidar_stick.urdf

File: cartographer_config/lidar_stick.urdf (robot description, URDF)
Before this commit: robot cartographer_backpack_3d, 3 links, 2 joints
Joints:
- joint gx5_link_joint: origin xyz=0 0 0 rpy=-1.57079632. 0 0 -> xyz=0 0 0 rpy=-1.57079632 0 0

Commit message: Update lidar_stick.urdf

File: cartographer_config/lidar_stick.urdf (robot description, URDF)
Before this commit: robot cartographer_backpack_3d, 3 links, 2 joints
Joints:
- joint gx5_link_joint: origin xyz=0 0 0 rpy=-1.57079632 0 0 -> xyz=0 0 0 rpy=0 1.57079632 1.5707632

Commit message: Update lidar_stick.urdf

File: cartographer_config/lidar_stick.urdf (robot description, URDF)
Before this commit: robot cartographer_backpack_3d, 3 links, 2 joints
Joints:
- joint gx5_link_joint: origin xyz=0 0 0 rpy=0 1.57079632 1.5707632 -> xyz=0 0 0 rpy=0 1.57079632 1.57079632

Commit message: Update lidar_stick.urdf

File: cartographer_config/lidar_stick.urdf (robot description, URDF)
Before this commit: robot cartographer_backpack_3d, 3 links, 2 joints
Joints:
- joint gx5_link_joint: origin xyz=0 0 0 rpy=0 1.57079632 1.57079632 -> xyz=0 0 0 rpy=3.14159265358979 -1.57079632 -1.57079632

Commit message: Update lidar_stick.urdf

File: cartographer_config/lidar_stick.urdf (robot description, URDF)
Before this commit: robot cartographer_backpack_3d, 3 links, 2 joints
Joints:
- joint velodyne_joint: origin xyz=0.030988 0 0.087378 rpy=0. 0 0 -> xyz=0 0.030988 0.087378 rpy=0. 0 0

Commit message: most significant minus sign ever, fixed the slam

File: cartographer_config/lidar_stick.urdf (robot description, URDF)
Before this commit: robot cartographer_backpack_3d, 3 links, 2 joints
Joints:
- joint gx5_link_joint: origin xyz=0 0 0 rpy=3.14159265358979 -1.57079632 -1.57079632 -> xyz=0 0 0 rpy=3.14159265358979 1.57079632 -1.57079632

Commit message: correct IMU orientation

File: cartographer_config/lidar_stick.urdf (robot description, URDF)
Before this commit: robot cartographer_backpack_3d, 3 links, 2 joints
Joints:
- joint velodyne_joint: origin xyz=0 0.030988 0.087378 rpy=0. 0 0 -> xyz=-0.030988 0 0.087378 rpy=0. 0 0

Commit message: this urdf is close to correct for the measurement taken on 01/18

File: cartographer_config/lidar_stick.urdf (robot description, URDF)
Before this commit: robot cartographer_backpack_3d, 3 links, 2 joints
Joints:
- joint velodyne_joint: origin xyz=-0.030988 0 0.087378 rpy=0. 0 0 -> xyz=0 0.030988 0.087378 rpy=0 0 4.75

Commit message: 1st guess with new mount

File: cartographer_config/lidar_stick.urdf (robot description, URDF)
Before this commit: robot cartographer_backpack_3d, 3 links, 2 joints
Joints:
- joint velodyne_joint: origin xyz=0 0.030988 0.087378 rpy=0 0 4.75 -> xyz=0 0.030988 0.072 rpy=0 0 3.14159265359

Commit message: 2nd guess

File: cartographer_config/lidar_stick.urdf (robot description, URDF)
Before this commit: robot cartographer_backpack_3d, 3 links, 2 joints
Joints:
- joint velodyne_joint: origin xyz=0 0.030988 0.072 rpy=0 0 3.14159265359 -> xyz=0 0.030988 0.072 rpy=0 0 -3.14159265359

Commit message: change to 0

File: cartographer_config/lidar_stick.urdf (robot description, URDF)
Before this commit: robot cartographer_backpack_3d, 3 links, 2 joints
Joints:
- joint velodyne_joint: origin xyz=0 0.030988 0.072 rpy=0 0 -3.14159265359 -> xyz=0 0.030988 0.072 rpy=0 0 0

Commit message: angle was 90 degrees off

File: cartographer_config/lidar_stick.urdf (robot description, URDF)
Before this commit: robot cartographer_backpack_3d, 3 links, 2 joints
Joints:
- joint velodyne_joint: origin xyz=0 0.030988 0.072 rpy=0 0 0 -> xyz=0 0.030988 0.072 rpy=0 0 1.57079632679
